File: pcb/headphone_dac/headphone_dac.kicad_pcb (KiCad board)
At the start: 2 copper layers, 75.5 x 62.5 mm, 69 parts, among them J1 USB_B_Mini, J2 Bluetooth, J3 Conn_01x05_Male, J6 Headphones, U1 LT3042xMSE, U2 CY8C5888LTI-LP097, U3 CS4344, U4 TPA6139A2, Y1 12.288MHz

Commit message: Add gerbers and schematics, update scripts
Other:
- rule pad_to_mask_clearance: 0.038 -> 0
